File: F3A_Board/F3A_Board.sch (KiCad schematic (older format))
At the start: 13 parts, among them J1 Conn_01x03, U1 LD1117AV33, U2 W25Q64V

Commit message: Eliminate blabla
Parts:
- removed C1: 100nF, Capacitor_THT:CP_Radial_D5.0mm_P2.50mm, symbol Device:C
- removed C2: 10uF, Capacitor_THT:CP_Radial_D5.0mm_P2.50mm, symbol Device:C
- removed U1: LD1117AV33, Package_TO_SOT_THT:TO-220-3_Vertical, symbol F3A_Modules:LD1117AV33
Changed lines of the file:
@@
 $EndComp
-$Comp
-L Device:C C1
-U 1 1 60996963
-P 4300 1400
-F 0 "C1" H 4415 1446 50  0000 L CNN
-F 1 "100nF" H 4415 1355 50  0000 L CNN
-F 2 "Capacitor_THT:CP_Radial_D5.0mm_P2.50mm" H 4338 1250 50  0001 C CNN
-F 3 "~" H 4300 1400 50  0001 C CNN
-	1    4300 1400
-	1    0    0    -1
-$EndComp
-$Comp
-L Device:C C2
-U 1 1 60997520
-P 5600 1400
-F 0 "C2" H 5715 1446 50  0000 L CNN
-F 1 "10uF" H 5715 1355 50  0000 L CNN
-F 2 "Capacitor_THT:CP_Radial_D5.0mm_P2.50mm" H 5638 1250 50  0001 C CNN
-F 3 "~" H 5600 1400 50  0001 C CNN
-	1    5600 1400
-	1    0    0    -1
-$EndComp
-$Comp
-L power:GND #PWR05
-U 1 1 60998C1D
-P 5000 1750
-F 0 "#PWR05" H 5000 1500 50  0001 C CNN
-F 1 "GND" H 5005 1577 50  0000 C CNN
-F 2 "" H 5000 1750 50  0001 C CNN
-F 3 "" H 5000 1750 50  0001 C CNN
-	1    5000 1750
-	1    0    0    -1
-$EndComp
-Wire Wire Line
-	5600 1550 5600 1650
-Wire Wire Line
-	4300 1650 4300 1550
-Wire Wire Line
-	4300 1650 5000 1650
-Wire Wire Line
-	5000 1750 5000 1650
-Connection ~ 5000 1650
-Wire Wire Line
-	5000 1650 5600 1650
-Wire Wire Line
-	4600 1100 4300 1100
-Wire Wire Line
-	4300 1100 4300 1250
-Wire Wire Line
-	5600 1100 5600 1250
-$Comp
-L power:+7.5V #PWR01
-U 1 1 6099A74A
-P 4050 1100
-F 0 "#PWR01" H 4050 950 50  0001 C CNN
-F 1 "+7.5V" V 4065 1228 50  0000 L CNN
-F 2 "" H 4050 1100 50  0001 C CNN
-F 3 "" H 4050 1100 50  0001 C CNN
-	1    4050 1100
-	0    -1   -1   0
-$EndComp
-$Comp
-L power:+3.3V #PWR07
-U 1 1 6099B91B
-P 5850 1100
-F 0 "#PWR07" H 5850 950 50  0001 C CNN
-F 1 "+3.3V" V 5865 1228 50  0000 L CNN
-F 2 "" H 5850 1100 50  0001 C CNN
-F 3 "" H 5850 1100 50  0001 C CNN
-	1    5850 1100
-	0    1    1    0
-$EndComp
-Wire Wire Line
-	5600 1100 5850 1100
-Wire Wire Line
-	5600 1100 5400 1100
-Connection ~ 5600 1100
-Wire Wire Line
-	4300 1100 4050 1100
-Connection ~ 4300 1100
 $Comp
 L power:+3.3V #PWR013
@@
 Text Label 1100 3300 2    50   ~ 0
 SPI3
-$Comp
-L F3A_Modules:LD1117AV33 U1
-U 1 1 609D4392
-P 5000 1200
-F 0 "U1" H 5000 1565 50  0000 C CNN
-F 1 "LD1117AV33" H 5000 1474 50  0000 C CNN
-F 2 "Package_TO_SOT_THT:TO-220-3_Vertical" H 5000 1150 50  0001 C CNN
-F 3 "" H 5000 1150 50  0001 C CNN
-	1    5000 1200
-	1    0    0    -1
-$EndComp
-Wire Wire Line
-	5000 1450 5000 1650
 Wire Wire Line
 	6750 3500 6750 3350
